Commit message: feat: mount sensor station on Bunker Pro 2

File: src/bunker_pro2/urdf/bunker_pro2.urdf (robot description, URDF)
Before this commit: robot bunker_pro2, 1 links, 0 joints
Links:
- added link sensor_station_link; visual mesh filename=package://bunker_pro2/meshes/FullCase.STL scale=0.001 0.001 0.001
Joints:
- added joint sensor_station_joint: type fixed, parent base_link, child sensor_station_link, origin xyz=-0.0075 0 0.016 rpy=0 0 0

Commit message: fix: align sensor station with physical mount

File: src/bunker_pro2/urdf/bunker_pro2.urdf (robot description, URDF)
Before this commit: robot bunker_pro2, 2 links, 1 joints
Joints:
- joint sensor_station_joint: origin xyz=-0.0075 0 0.016 rpy=0 0 0 -> xyz=-0.0075 0 0.016 rpy=1.57079632679 0 3.14159265359

Commit message: feat: add sensor station camera TF

File: src/bunker_pro2/urdf/bunker_pro2.urdf (robot description, URDF)
Before this commit: robot bunker_pro2, 2 links, 1 joints
Links:
- added link camera_link
Joints:
- added joint sensor_station_camera_joint: type fixed, parent sensor_station_link, child camera_link, origin xyz=0.2212 0 0.318 rpy=0 0 0

Commit message: fix: save calibrated sensor and camera transforms

File: src/bunker_pro2/urdf/bunker_pro2.urdf (robot description, URDF)
Before this commit: robot bunker_pro2, 3 links, 2 joints
Joints:
- joint sensor_station_camera_joint: origin xyz=0.2212 0 0.318 rpy=0 0 0 -> xyz=-0.2212 0.318 0 rpy=1.57079632679 0 3.14159265359
- joint sensor_station_joint: origin xyz=-0.0075 0 0.016 rpy=1.57079632679 0 3.14159265359 -> xyz=-0.2125 0 0.016 rpy=1.57079632679 0 3.14159265359

Commit message: feat: add calibrated LiDAR TF

File: src/bunker_pro2/urdf/bunker_pro2.urdf (robot description, URDF)
Before this commit: robot bunker_pro2, 3 links, 2 joints
Links:
- added link lidar_link
Joints:
- added joint sensor_station_lidar_joint: type fixed, parent sensor_station_link, child lidar_link, origin xyz=0 0.4 0 rpy=1.57079632679 0 3.14159265359

Commit message: feat(bunker-pro2): add physical robot TF description

File: src/bunker_pro2/urdf/bunker_pro2.urdf (robot description, URDF)
Before this commit: robot bunker_pro2, 4 links, 3 joints
Links:
- added link robot_bottom
Joints:
- added joint robot_bottom_to_base_link: type fixed, parent robot_bottom, child base_link, origin xyz=0 0 0.45 rpy=0 0 0

Commit message: fix(tf): define canonical camera reference chain

File: src/bunker_pro2/urdf/bunker_pro2.urdf (robot description, URDF)
Before this commit: robot bunker_pro2, 5 links, 4 joints
Links:
- added link camera_mount_link
- added link zed_camera_link
Joints:
- removed joint sensor_station_camera_joint
- added joint camera_mount_to_camera_joint: type fixed, parent camera_mount_link, child camera_link, origin xyz=-0.185 0 0 rpy=0 0 0
- added joint camera_to_zed_camera_joint: type fixed, parent camera_link, child zed_camera_link, origin xyz=0.01 0 -0.015 rpy=0 0 0
- added joint sensor_station_camera_mount_joint: type fixed, parent sensor_station_link, child camera_mount_link, origin xyz=-0.2212 0.318 0 rpy=1.57079632679 0 3.14159265359

Commit message: fix(tf): align camera mount with stereo center

File: src/bunker_pro2/urdf/bunker_pro2.urdf (robot description, URDF)
Before this commit: robot bunker_pro2, 7 links, 6 joints
Links:
- removed link camera_link
Joints:
- removed joint camera_mount_to_camera_joint
- removed joint camera_to_zed_camera_joint
- added joint camera_mount_to_zed_camera_joint: type fixed, parent camera_mount_link, child zed_camera_link, origin xyz=0 0 -0.015 rpy=0 0 0

Commit message: feat(tf): attach PiPER arm to Bunker front rail

File: src/bunker_pro2/urdf/bunker_pro2.urdf (robot description, URDF)
Before this commit: robot bunker_pro2, 6 links, 5 joints
Links:
- added link arm_base_link, mass 1.02; collision mesh filename=package://piper_description/meshes/base_link.STL; visual mesh filename=package://piper_description/meshes/base_link.STL
- added link camera_holder; visual mesh filename=package://piper_description/meshes/camera_holder.STL scale=0.001 0.001 0.001
- added link gripper_base, mass 0.45; collision mesh filename=package://piper_description/meshes/gripper_base.STL; visual mesh filename=package://piper_description/meshes/gripper_base.STL
- added link l515_visual; visual mesh filename=package://piper_description/meshes/Intel_RealSense_L515_CAD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 scale=0.001 0.001 0.001
- added link link1, mass 0.71; collision mesh filename=package://piper_description/meshes/link1.STL; visual mesh filename=package://piper_description/meshes/link1.STL
- added link link2, mass 1.17; collision mesh filename=package://piper_description/meshes/link2.STL; visual mesh filename=package://piper_description/meshes/link2.STL
- added link link3, mass 0.5; collision mesh filename=package://piper_description/meshes/link3.STL; visual mesh filename=package://piper_description/meshes/link3.STL
- added link link4, mass 0.38; collision mesh filename=package://piper_description/meshes/link4.STL; visual mesh filename=package://piper_description/meshes/link4.STL
- added link link5, mass 0.383; collision mesh filename=package://piper_description/meshes/link5.STL; visual mesh filename=package://piper_description/meshes/link5.STL
- added link link6, mass 0.00699089613564366; collision mesh filename=package://piper_description/meshes/link6.STL; visual mesh filename=package://piper_description/meshes/link6.STL
- added link link7, mass 0.025; collision mesh filename=package://piper_description/meshes/link7.STL; visual mesh filename=package://piper_description/meshes/link7.STL
- added link link8, mass 0.025; collision mesh filename=package://piper_description/meshes/link8.STL; visual mesh filename=package://piper_description/meshes/link8.STL
Joints:
- added joint base_to_arm_base_joint: type fixed, parent base_link, child arm_base_link, origin xyz=0.39 0 0.016 rpy=0 0 0
- added joint camera_holder_to_l515_visual: type fixed, parent camera_holder, child l515_visual, origin xyz=0.1 0 0 rpy=-3.141592653589793  3.141592653589793 1.5707963267948966
- added joint gripper_base_to_camera_holder: type fixed, parent gripper_base, child camera_holder, origin xyz=-0.036 0 0.044 rpy=0 0 0
- added joint joint1: type revolute, parent arm_base_link, child link1, origin xyz=0 0 0.123 rpy=0 0 0, axis 0 0 1, limit lower=-2.618 upper=2.168 effort=100 velocity=5
- added joint joint2: type revolute, parent link1, child link2, origin xyz=0 0 0 rpy=1.5707963267948966 -0.10088003076527219 -3.141592653589793, axis 0 0 1, limit lower=-0.044796192 upper=3.14 effort=100 velocity=5
- added joint joint3: type revolute, parent link2, child link3, origin xyz=0.28503 0 0 rpy=0 0 -1.7589428201598853, axis 0 0 1, limit lower=-2.967 upper=0 effort=100 velocity=5
- added joint joint4: type revolute, parent link3, child link4, origin xyz=-0.02198 -0.25075 0 rpy=1.5707963267948966 0 0, axis 0 0 1, limit lower=-1.745 upper=1.745 effort=100 velocity=5
- added joint joint5: type revolute, parent link4, child link5, origin xyz=0 0 0 rpy=-1.5707963267948966 0 0, axis 0 0 1, limit lower=-1.22 upper=1.22 effort=100 velocity=5
- added joint joint6: type revolute, parent link5, child link6, origin xyz=0 -0.091 0 rpy=1.5707963267948966 0 0, axis 0 0 1, limit lower=-2.0944 upper=2.0944 effort=100 velocity=3
- added joint joint6_to_gripper_base: type fixed, parent link6, child gripper_base, origin xyz=0 0 0 rpy=0 0 3.141592653589793
- added joint joint7: type prismatic, parent gripper_base, child link7, origin xyz=0 0 0.1358 rpy=1.5708 0 0, axis 0 0 1, limit lower=0 upper=0.035 effort=10 velocity=1
- added joint joint8: type prismatic, parent gripper_base, child link8, origin xyz=0 0 0.1358 rpy=1.5708 0 -3.1416, axis 0 0 -1, limit lower=-0.035 upper=0 effort=10 velocity=1
